File: bottom plate.kicad_pcb (KiCad board)
At the start: 2 copper layers, 190.5 x 76.2 mm, 5 parts

Commit message: gerbs updated and stuff
Parts:
- added REF**: M2_Hole_NPTH_Outside, kbd:M2_Hole_NPTH_Outside, F.Cu at (61.1, 31.8)
Other:
- board text added: "JLCJLCJLCJLC"
Changed lines of the file:
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@@
   (general
     (thickness 1.6)
-    (drawings 8)
+    (drawings 9)
     (tracks 0)
     (zones 0)
-    (modules 5)
+    (modules 6)
     (nets 1)
   )
@@
     (uvia_drill 0.1)
   )
+  (module kbd:M2_Hole_NPTH_Outside (layer F.Cu)
+    (at 61.11875 31.75)
+    (fp_text reference REF** (at 0 0.5) (layer F.SilkS) hide
+      (effects (font (size 1 1) (thickness 0.15)))
+    )
+    (fp_text value M2_Hole_NPTH_Outside (at 0 -0.5) (layer F.Fab)
+      (effects (font (size 1 1) (thickness 0.15)))
+    )
+    (pad "" np_thru_hole circle (at 0 0) (size 4 4) (drill 4) (layers *.Cu *.Mask))
+  )
   (module kbd:M2_HOLE_v3 (layer F.Cu)
     (at 114.3 55.5625)
@@
     (pad 1 thru_hole circle (at 0 0) (size 4 4) (drill 2.3) (layers *.Cu *.Mask))
   )
+  (gr_text JLCJLCJLCJLC (at 114.3 50.8) (layer F.SilkS)
+    (effects (font (size 1 1) (thickness 0.15)))
+  )
   (gr_line (start 207.9625 17.4625) (end 20.6375 17.4625) (layer Edge.Cuts) (width 0.05))
