File: cheapcheep.kicad_pcb (KiCad board)
At the start: 2 copper layers, 190.5 x 76.2 mm, 95 parts, among them SW1 SW_Push, U1 ProMicro

Commit message: gerbs updated and stuff
Other:
- board text added: "JLCJLCJLCJLC"
Changed lines of the file:
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@@
   (general
     (thickness 1.6)
-    (drawings 694)
+    (drawings 695)
     (tracks 359)
     (zones 0)
@@
     (pad "" np_thru_hole circle (at 5.08 0 48.0996) (size 1.75 1.75) (drill 1.75) (layers *.Cu *.Mask))
   )
+  (gr_text JLCJLCJLCJLC (at 114.3 52.3875) (layer B.SilkS)
+    (effects (font (size 1 1) (thickness 0.15)) (justify mirror))
+  )
   (gr_arc (start 47.350902 34.677683) (end 49.432256 38.824861) (angle -10.21388279) (layer B.SilkS) (width 0.02))
